Commit message: feat: Update package name

File: catkin_ws/src/slam_project/urdf/hsin_bot.xacro (robot description, xacro)
@@ -1,5 +1,5 @@
 <?xml version='1.0'?>
-<robot name="udacity_bot" xmlns:xacro="http://www.ros.org/wiki/xacro">
-  <xacro:include filename="$(find udacity_bot)/urdf/hsin_bot.gazebo" />
+<robot name="hsin_bot" xmlns:xacro="http://www.ros.org/wiki/xacro">
+  <xacro:include filename="$(find slam_project)/urdf/hsin_bot.gazebo" />
   <link name="robot_footprint"></link>
   <joint name="robot_footprint_joint" type="fixed">
@@ -204,5 +204,5 @@
       <origin xyz="0.0 0 0" rpy=" 0 0 0"/>
       <geometry>
-        <mesh filename="package://udacity_bot/meshes/hokuyo.dae"/>
+        <mesh filename="package://slam_project/meshes/hokuyo.dae"/>
       </geometry>
     </visual>

Commit message: Fix: TF of received image 0 at time 180.464000s is not set!
Add camera_rgbd_frame

File: catkin_ws/src/slam_project/urdf/hsin_bot.xacro (robot description, xacro)
@@ -185,4 +185,10 @@
     <dynamics damping="1.0" friction="1.0"/>
   </joint>
+  <link name="camera_rgbd_frame"></link>
+  <joint name="camera_rgbd_joint" type="fixed">
+    <origin xyz="0 0 0" rpy="-${pi/2} 0 -${pi/2}"/>
+    <parent link="camera"/>
+    <child link="camera_rgbd_frame"/>
+  </joint>
   <link name="hokuyo">
     <inertial>
